File: PCB/SpiritBall-Debug.kicad_sch (KiCad schematic)
At the start: 6 parts

Commit message: Version 0.3.0, sent for fabrication
Parts:
- D37, D38: value (none) -> 1N5819HW-7-F; footprint (none) -> Diode_SMD:D_SOD-123
- J2: value (none) -> TAG_CONNECT_JTAG; footprint (none) -> Connector:Tag-Connect_TC2050-IDC-FP_2x05_P1.27mm_Vertical
- J3: value (none) -> HEADER_DBG; footprint (none) -> Connector_PinHeader_1.27mm:PinHeader_2x03_P1.27mm_Vertical
- J4: value (none) -> HEADER_JTAG; footprint (none) -> Connector_PinHeader_1.27mm:PinHeader_2x05_P1.27mm_Vertical
- J5: value (none) -> TAG_CONNECT_DBG; footprint (none) -> Connector:Tag-Connect_TC2030-IDC-FP_2x03_P1.27mm_Vertical
Connections:
- net USB_5V: now also D37.1, D38.1; no longer D37.C, D38.C
- net at J3.2 (VCC), J5.2 (VCC): now also D38.2; no longer D38.A
- net at J2.1 (VCC), J4.1 (VCC): now also D37.2; no longer D37.A
Changed lines of the file:
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@@
       (effects (font (size 1.27 1.27)) (justify right))
     )
-    (property "Value" "" (id 1) (at 91.44 129.54 0)
+    (property "Value" "HEADER_DBG" (id 1) (at 87.63 129.54 0)
       (effects (font (size 1.27 1.27)) (justify right))
     )
-    (property "Footprint" "" (id 2) (at 69.85 140.97 90)
+    (property "Footprint" "Connector_PinHeader_1.27mm:PinHeader_2x03_P1.27mm_Vertical" (id 2) (at 69.85 140.97 90)
       (effects (font (size 1.27 1.27)) hide)
     )
@@
     (in_bom yes) (on_board yes) (fields_autoplaced)
     (property "Reference" "D38" (id 0) (at 128.27 114.3 0))
-    (property "Value" "" (id 1) (at 128.27 116.84 0))
-    (property "Footprint" "" (id 2) (at 128.27 120.65 0)
+    (property "Value" "1N5819HW-7-F" (id 1) (at 128.27 116.84 0))
+    (property "Footprint" "Diode_SMD:D_SOD-123" (id 2) (at 128.27 120.65 0)
       (effects (font (size 1.27 1.27)) (justify left bottom) hide)
     )
@@
       (effects (font (size 1.27 1.27)) (justify left bottom) hide)
     )
-    (pin "A")
-    (pin "C")
+    (pin "1")
+    (pin "2")
   )
-  (symbol (lib_id "MyParts:1N5819HW-7-F") (at 128.27 43.18 0) (unit 1)
-    (in_bom yes) (on_board yes) (fields_autoplaced)
+  (symbol (lib_name "1N5819HW-7-F_1") (lib_id "MyParts:1N5819HW-7-F") (at 128.27 43.18 0) (unit 1)
+    (in_bom yes) (on_board yes)
     (property "Reference" "D37" (id 0) (at 128.27 36.83 0))
-    (property "Value" "" (id 1) (at 128.27 39.37 0))
-    (property "Footprint" "" (id 2) (at 128.27 43.18 0)
+    (property "Value" "1N5819HW-7-F" (id 1) (at 128.27 39.37 0))
+    (property "Footprint" "Diode_SMD:D_SOD-123" (id 2) (at 128.27 43.18 0)
       (effects (font (size 1.27 1.27)) (justify left bottom) hide)
     )
@@
       (effects (font (size 1.27 1.27)) (justify left bottom) hide)
     )
-    (pin "A")
-    (pin "C")
+    (pin "1")
+    (pin "2")
   )
   (symbol (lib_id "MyParts:ESP-PROG-JTAG-1.27") (at 113.03 64.77 0) (unit 1)
@@
       (effects (font (size 1.27 1.27)) (justify right))
     )
-    (property "Value" "" (id 1) (at 134.62 53.34 0)
+    (property "Value" "HEADER_JTAG" (id 1) (at 124.46 53.34 0)
       (effects (font (size 1.27 1.27)) (justify right))
     )
-    (property "Footprint" "" (id 2) (at 109.22 60.96 90)
+    (property "Footprint" "Connector_PinHeader_1.27mm:PinHeader_2x05_P1.27mm_Vertical" (id 2) (at 109.22 60.96 90)
       (effects (font (size 1.27 1.27)) hide)
     )
@@
       (effects (font (size 1.27 1.27)) (justify right))
     )
-    (property "Value" "" (id 1) (at 96.52 53.34 0)
+    (property "Value" "TAG_CONNECT_JTAG" (id 1) (at 92.71 53.34 0)
       (effects (font (size 1.27 1.27)) (justify right))
     )
-    (property "Footprint" "" (id 2) (at 71.12 60.96 90)
+    (property "Footprint" "Connector:Tag-Connect_TC2050-IDC-FP_2x05_P1.27mm_Vertical" (id 2) (at 71.12 60.96 90)
       (effects (font (size 1.27 1.27)) hide)
     )
@@
       (effects (font (size 1.27 1.27)) (justify right))
     )
-    (property "Value" "" (id 1) (at 134.62 129.54 0)
+    (property "Value" "TAG_CONNECT_DBG" (id 1) (at 135.89 129.54 0)
       (effects (font (size 1.27 1.27)) (justify right))
     )
-    (property "Footprint" "" (id 2) (at 113.03 140.97 90)
+    (property "Footprint" "Connector:Tag-Connect_TC2030-IDC-FP_2x03_P1.27mm_Vertical" (id 2) (at 113.03 140.97 90)
       (effects (font (size 1.27 1.27)) hide)
     )
