File: PCB/SpiritBall-LEDs.kicad_sch (KiCad schematic)
At the start: 35 parts

Commit message: Version 0.3.0, sent for fabrication
Parts:
- added C6: 1000uF, Capacitor_SMD:C_Elec_8x10.2, symbol Device:C_Polarized_Small_US
Connections:
- net LED Ground: now also C6.2
- net LED Power: now also C6.1
Changed lines of the file:
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@@
+    (stroke (width 0) (type default) (color 0 0 0 0))
+  )
+  (wire (pts (xy 237.49 39.37) (xy 237.49 44.45))
     (stroke (width 0) (type default) (color 0 0 0 0))
   )
@@
     (stroke (width 0) (type default) (color 0 0 0 0))
   )
+  (wire (pts (xy 237.49 29.21) (xy 237.49 34.29))
+    (stroke (width 0) (type default) (color 0 0 0 0))
+  )
   (wire (pts (xy 50.8 67.31) (xy 55.88 67.31))
     (stroke (width 0) (type default) (color 0 0 0 0))
@@
     (stroke (width 0) (type default) (color 0 0 0 0))
   )
+  (hierarchical_label "LED Ground" (shape input) (at 237.49 44.45 180)
+    (effects (font (size 1.27 1.27)) (justify right))
+  )
   (hierarchical_label "LED Data IN" (shape input) (at 48.26 33.02 180)
     (effects (font (size 1.27 1.27)) (justify right))
   )
   (hierarchical_label "LED Power" (shape input) (at 125.73 53.34 180)
+    (effects (font (size 1.27 1.27)) (justify right))
+  )
+  (hierarchical_label "LED Power" (shape input) (at 237.49 29.21 180)
     (effects (font (size 1.27 1.27)) (justify right))
   )
@@
     (pin "4")
   )
+  (symbol (lib_id "Device:C_Polarized_Small_US") (at 237.49 36.83 0) (unit 1)
+    (in_bom yes) (on_board yes) (fields_autoplaced)
+    (property "Reference" "C6" (id 0) (at 240.03 35.1281 0)
+      (effects (font (size 1.27 1.27)) (justify left))
+    )
+    (property "Value" "1000uF" (id 1) (at 240.03 37.6681 0)
+      (effects (font (size 1.27 1.27)) (justify left))
+    )
+    (property "Footprint" "Capacitor_SMD:C_Elec_8x10.2" (id 2) (at 237.49 36.83 0)
+      (effects (font (size 1.27 1.27)) hide)
+    )
+    (property "Datasheet" "~" (id 3) (at 237.49 36.83 0)
+      (effects (font (size 1.27 1.27)) hide)
+    )
+    (pin "1")
+    (pin "2")
+  )
   (symbol (lib_id "LED:WS2812B") (at 114.3 33.02 0) (unit 1)
