File: PCB/SpiritBall-S3.kicad_sch (KiCad schematic)
At the start: 17 parts, among them J1 105450-0101, SW1 SW_Push, U1 ESP32-S3-WROOM-1, U2 AZ1117CD-3.3TRG1

Commit message: Version 0.3.0, sent for fabrication
Parts:
- removed D39, D40, D41: LESD5D5.0CT1G, MyParts:TVS_LESD5D5.0CT1G, symbol MyParts:LESD5D5.0CT1G
- removed SW1: SW_Push, Button_Switch_SMD:SW_SPST_B3S-1000, symbol Switch:SW_Push
- added D39, D40, D41: LESD5Z5.0CT1G, Diode_SMD:D_SOD-523, symbol MyParts:LESD5Z5.0CT1G
- added R5: 10K, Resistor_SMD:R_0402_1005Metric, symbol Device:R
- added SW1, SW2: TS-1187A-B-A-B, MyParts:SW_TS-1187A-B-A-B, symbol MyParts:TS-1187A-B-A-B
- C1: value 1uF/16V(10%) -> 1uF
- C2: value 10uF/25V(20%) -> 10uF
- C3: value 0.1uF/50V(10%) -> 0.1uF
- D36: footprint MyParts:SOD3715X145N -> Diode_SMD:D_SOD-123
- R1: value 10K(1%) -> 10K
- R2: value 0(1%) -> 0k
- R3, R4: value 5.1k(10%) -> 5.1k
Connections:
- net +3.3V: now also R5.2
- net +5V: now also D36.1; no longer D36.C
- net EN/CHIP_PU: now also SW1.A, SW1.B
- net GND: now also D39.1, D40.1, D41.1, SW1.C, SW1.D, SW2.C, SW2.D
- net USB_D+: now also D40.2
- net USB_D-: now also D41.2
- net at U1.10 (GPIO17/U1TXD/ADC2_CH6): now also R5.1, SW2.A, SW2.B
- net at J1.A4 (VBUS_A), J1.A9 (VBUS_A), J1.B4 (VBUS_B)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: now also D36.2, D39.2; no longer D36.A
