File: PCB/SpiritBall.kicad_pcb (KiCad board)
At the start: 4 copper layers, 100 x 100 mm, 59 parts, among them J1 105450-0101, J2 ESP-PROG-JTAG-1.27, J3 ESP-PROG-1.27, J4 ESP-PROG-JTAG-1.27, J5 ESP-PROG-1.27, SW1 SW_Push, U1 ESP32-S3-WROOM-1, U2 AZ1117CD-3.3TRG1

Commit message: Version 0.3.0, sent for fabrication
Parts:
- added C6: 1000uF, Capacitor_SMD:C_Elec_8x10.2, F.Cu at (75.6, 84.5)
- added R5: 10K, Resistor_SMD:R_0402_1005Metric, F.Cu at (112.5, 96.1)
- added SW2: TS-1187A-B-A-B, MyParts:SW_TS-1187A-B-A-B, F.Cu at (119.2, 91.0)
- C1: value 1uF/16V(10%) -> 1uF
- C2: value 10uF/25V(20%) -> 10uF
- C3: value 0.1uF/50V(10%) -> 0.1uF
- D36, D37, D38: footprint MyParts:SOD3715X145N -> Diode_SMD:D_SOD-123
- D39, D40, D41: value LESD5D5.0CT1G -> LESD5Z5.0CT1G; footprint MyParts:TVS_LESD5D5.0CT1G -> Diode_SMD:D_SOD-523
- J2: value ESP-PROG-JTAG-1.27 -> TAG_CONNECT_JTAG
- J3: value ESP-PROG-1.27 -> HEADER_DBG
- J4: value ESP-PROG-JTAG-1.27 -> HEADER_JTAG
- J5: value ESP-PROG-1.27 -> TAG_CONNECT_DBG
- R1: value 10K(1%) -> 10K
- R2: value 0(1%) -> 0k
- R3, R4: value 5.1k(10%) -> 5.1k
- SW1: value SW_Push -> TS-1187A-B-A-B; footprint Button_Switch_SMD:SW_SPST_B3S-1000 -> MyParts:SW_TS-1187A-B-A-B
- moved SW1 0.42 mm to (119.2, 98.7)
Connections:
- D39 pad 2: Net-(D36-PadA) -> Net-(D36-Pad2)
- J1 pad A4: Net-(D36-PadA) -> Net-(D36-Pad2)
- J1 pad A9: Net-(D36-PadA) -> Net-(D36-Pad2)
- J1 pad B4: Net-(D36-PadA) -> Net-(D36-Pad2)
- J1 pad B9: Net-(D36-PadA) -> Net-(D36-Pad2)
- J2 pad 1: Net-(D37-PadA) -> Net-(D37-Pad2)
- J3 pad 2: Net-(D38-PadA) -> Net-(D38-Pad2)
- J4 pad 1: Net-(D37-PadA) -> Net-(D37-Pad2)
- J5 pad 2: Net-(D38-PadA) -> Net-(D38-Pad2)
- U1 pad 10: unconnected-(U1-Pad10) -> Net-(R5-Pad1)
Routing:
- net Net-(R5-Pad1): track 0.00 -> 17.1 mm
- net Net-(D37-PadA): track 14.6 -> 0.00 mm
- net Net-(D37-Pad2): track 0.00 -> 14.6 mm
- net Net-(D38-PadA): track 14.1 -> 0.00 mm
- net Net-(D38-Pad2): track 0.00 -> 14.1 mm
- net Net-(D36-PadA): track 13.2 -> 0.00 mm
- net Net-(D36-Pad2): track 0.00 -> 13.2 mm
- net GND: track 176.9 -> 186.4 mm, vias 44 -> 46
- net +5V: track 143.1 -> 147.1 mm, vias 39 -> 40
- net EN/CHIP_PU: track 60.0 -> 62.3 mm
- net +3.3V: track 11.4 -> 12.7 mm, vias 1 -> 2
Other:
- board text added: "Brendon McCool SpiritBall V0.3.1 2022-10-20 JLCJLCJLCJLC"
